File: thumbs-down-hw/thumbs-down-hw.kicad_pcb (KiCad board)
At the start: 2 copper layers, 28.2 x 97.2 mm, 26 parts, among them SW10 SW_Push, SW2 SW_Push, SW3 SW_Push, SW9 SW_Push, U1 PicoW, U2 RFM69HCW

Commit message: rename thumbs-down-hw
Routing:
- net GND: track 88.5 -> 98.6 mm, vias 49 -> 53
Other:
- board text added: "ihartwig ©2023 r1"
- board text added: "thumbs-down dev kit"
Changed lines of the file:
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@@
     (property "ki_keywords" "Adafruit feather microcontroller module")
     (attr through_hole)
-    (fp_text reference "A1" (at 10.16 -7.62) (layer "F.SilkS")
+    (fp_text reference "A1" (at 2.794 -8.001 90) (layer "F.SilkS")
         (effects (font (size 1 1) (thickness 0.15)))
     )
@@
     (property "ki_keywords" "low power Radio ISM Transceiver Module AES encryption SPI HopeRF")
     (attr smd)
-    (fp_text reference "U2" (at 0 -9.2 90) (layer "F.SilkS")
+    (fp_text reference "U2" (at 0 -9.017 90) (layer "F.SilkS")
         (effects (font (size 1 1) (thickness 0.15)))
     )
@@
       (net 20 "+5V") (pinfunction "VBUS") (pintype "unspecified"))
   )
+  (gr_line (start 139.954 92.583) (end 139.954 92.075)
+    (stroke (width 0.15) (type default)) (layer "F.SilkS"))
   (gr_arc (start 135.255 50.165) (mid 136.184934 47.919932) (end 138.43 46.99)
     (stroke (width 0.1) (type default)) (layer "Edge.Cuts"))
@@
   (gr_line (start 138.43 46.99) (end 151.765 46.99)
     (stroke (width 0.1) (type default)) (layer "Edge.Cuts"))
+  (gr_text "thumbs-down dev kit" (at 138.557 62.992 90) (layer "B.Cu")
+    (effects (font (size 1 0.9) (thickness 0.1524)) (justify left bottom mirror))
+  )
+  (gr_text "ihartwig  ©2023  r1" (at 137.033 61.849 90) (layer "B.Cu")
+    (effects (font (size 1 1) (thickness 0.1524)) (justify left bottom mirror))
+  )
   (gr_text "SDA" (at 153.035 137.16 315) (layer "F.SilkS")
     (effects (font (size 0.8 0.8) (thickness 0.15)))
@@
   (segment (start 152.1968 65.093) (end 152.1968 65.2526) (width 0.2032) (layer "F.Cu") (net 2))
   (segment (start 156.845 70.485) (end 157.48 71.12) (width 0.6096) (layer "F.Cu") (net 2))
+  (segment (start 157.988 79.502) (end 157.353 78.867) (width 0.2032) (layer "F.Cu") (net 2))
   (segment (start 136.652 92.71) (end 139.192 92.71) (width 0.3048) (layer "F.Cu") (net 2))
   (segment (start 143.891 128.27) (end 144.526 128.905) (width 0.2032) (layer "F.Cu") (net 2))
@@
   (segment (start 156.845 83.185) (end 157.48 82.55) (width 0.6096) (layer "F.Cu") (net 2))
   (segment (start 162.56 83.82) (end 162.56 85.09) (width 0.6096) (layer "F.Cu") (net 2))
+  (segment (start 157.988 80.518) (end 157.988 79.502) (width 0.2032) (layer "F.Cu") (net 2))
+  (segment (start 155.194 78.486) (end 155.194 79.375) (width 0.2032) (layer "F.Cu") (net 2))
+  (segment (start 155.575 73.025) (end 155.194 73.025) (width 0.6096) (layer "F.Cu") (net 2))
   (segment (start 161.8488 66.5988) (end 161.8488 65.4232) (width 0.6096) (layer "F.Cu") (net 2))
   (segment (start 141.971 104.125) (end 142.367 104.521) (width 0.6096) (layer "F.Cu") (net 2))
@@
   (segment (start 153.971 86.059) (end 154.94 85.09) (width 0.6096) (layer "F.Cu") (net 2))
   (segment (start 155.971 104.633) (end 155.1686 105.4354) (width 0.6096) (layer "F.Cu") (net 2))
+  (segment (start 155.575 78.867) (end 155.194 78.486) (width 0.2032) (layer "F.Cu") (net 2))
   (segment (start 153.1112 65.093) (end 153.1112 66.7512) (width 0.6096) (layer "F.Cu") (net 2))
   (segment (start 160.02 87.63) (end 159.385 88.265) (width 0.6096) (layer "F.Cu") (net 2))
   (segment (start 146.685 84.455) (end 147.066 84.836) (width 0.2032) (layer "F.Cu") (net 2))
+  (segment (start 157.353 78.867) (end 155.575 78.867) (width 0.2032) (layer "F.Cu") (net 2))
   (segment (start 143.825 113.03) (end 143.891 113.03) (width 0.2032) (layer "F.Cu") (net 2))
   (segment (start 143.891 125.73) (end 144.526 125.095) (width 0.2032) (layer "F.Cu") (net 2))
@@
   (segment (start 143.825 125.73) (end 143.891 125.73) (width 0.2032) (layer "F.Cu") (net 2))
   (segment (start 152.1968 65.2526) (end 151.9174 65.532) (width 0.2032) (layer "F.Cu") (net 2))
+  (segment (start 157.48 81.28) (end 157.48 81.026) (width 0.2032) (layer "F.Cu") (net 2))
   (segment (start 162.56 68.58) (end 162.56 69.85) (width 0.6096) (layer "F.Cu") (net 2))
   (segment (start 141.971 101.361) (end 142.367 100.965) (width 0.6096) (layer "F.Cu") (net 2))
   (segment (start 152.715 119.314) (end 153.035 119.634) (width 0.3048) (layer "F.Cu") (net 2))
+  (segment (start 157.48 71.12) (end 155.575 73.025) (width 0.6096) (layer "F.Cu") (net 2))
   (segment (start 139.954 106.68) (end 141.351 106.68) (width 0.3048) (layer "F.Cu") (net 2))
   (segment (start 143.825 115.57) (end 143.891 115.57) (width 0.2032) (layer "F.Cu") (net 2))
@@
   (segment (start 136.652 105.41) (end 137.922 106.68) (width 0.3048) (layer "F.Cu") (net 2))
   (segment (start 154.305 67.945) (end 154.94 68.58) (width 0.6096) (layer "F.Cu") (net 2))
+  (segment (start 157.48 81.026) (end 157.988 80.518) (width 0.2032) (layer "F.Cu") (net 2))
   (segment (start 141.971 102.775) (end 141.971 104.125) (width 0.6096) (layer "F.Cu") (net 2))
   (segment (start 142.555 71.755) (end 142.555 71.943) (width 0.2032) (layer "F.Cu") (net 2))
@@
   (via (at 154.94 85.09) (size 0.6096) (drill 0.3048) (layers "F.Cu" "B.Cu") (net 2))
   (via (at 162.56 77.47) (size 0.6096) (drill 0.3048) (layers "F.Cu" "B.Cu") (net 2))
+  (via (at 155.194 79.375) (size 0.6096) (drill 0.3048) (layers "F.Cu" "B.Cu") (net 2))
   (via (at 159.385 88.265) (size 0.6096) (drill 0.3048) (layers "F.Cu" "B.Cu") (net 2))
   (via (at 156.21 69.85) (size 0.6096) (drill 0.3048) (layers "F.Cu" "B.Cu") (net 2))
@@
   (via (at 144.526 116.205) (size 0.6096) (drill 0.3048) (layers "F.Cu" "B.Cu") (net 2))
   (via (at 156.845 83.185) (size 0.6096) (drill 0.3048) (layers "F.Cu" "B.Cu") (net 2))
+  (via (at 155.194 78.486) (size 0.6096) (drill 0.3048) (layers "F.Cu" "B.Cu") (net 2))
   (via (at 162.56 68.58) (size 0.6096) (drill 0.3048) (layers "F.Cu" "B.Cu") (net 2))
   (via (at 162.56 74.93) (size 0.6096) (drill 0.3048) (layers "F.Cu" "B.Cu") (net 2))
@@
   (via (at 162.56 83.82) (size 0.6096) (drill 0.3048) (layers "F.Cu" "B.Cu") (net 2))
   (via (at 162.56 69.85) (size 0.6096) (drill 0.3048) (layers "F.Cu" "B.Cu") (net 2))
+  (via (at 155.194 73.025) (size 0.6096) (drill 0.3048) (layers "F.Cu" "B.Cu") (net 2))
   (via (at 145.161 75.819) (size 0.6096) (drill 0.3048) (layers "F.Cu" "B.Cu") (net 2))
   (via (at 157.48 82.55) (size 0.6096) (drill 0.3048) (layers "F.Cu" "B.Cu") (net 2))
@@
   (via (at 162.56 67.31) (size 0.6096) (drill 0.3048) (layers "F.Cu" "B.Cu") (net 2))
   (via (at 161.925 85.725) (size 0.6096) (drill 0.3048) (layers "F.Cu" "B.Cu") (net 2))
+  (via (at 155.194 73.914) (size 0.6096) (drill 0.3048) (layers "F.Cu" "B.Cu") (net 2))
   (via (at 160.655 86.995) (size 0.6096) (drill 0.3048) (layers "F.Cu" "B.Cu") (net 2))
   (segment (start 156.21 83.82) (end 156.845 83.185) (width 0.6096) (layer "B.Cu") (net 2))
@@
   (segment (start 162.56 80.01) (end 162.56 81.28) (width 0.6096) (layer "B.Cu") (net 2))
   (segment (start 155.194 105.41) (end 155.1686 105.4354) (width 0.6096) (layer "B.Cu") (net 2))
+  (segment (start 155.194 73.025) (end 155.194 73.914) (width 0.6096) (layer "B.Cu") (net 2))
   (segment (start 157.48 82.55) (end 157.48 81.28) (width 0.6096) (layer "B.Cu") (net 2))
   (segment (start 161.29 86.36) (end 160.655 86.995) (width 0.6096) (layer "B.Cu") (net 2))

Commit message: add thumbs-down-hw r1 gerbers
Parts:
- moved C4 19.1 mm to (142.9, 128.3)
- moved C3 10.2 mm to (142.9, 115.6)
- moved C1 6.35 mm to (142.9, 109.2)
- moved C5 2.54 mm to (142.9, 125.7)
- renumbered D2 to D1, SW2 to SW1
Connections:
- net /LED_DI_2 renamed /LED_DI_3
- A1 pad 19: /GPIO2 -> /GPIO3
- A1 pad 20: /GPIO10 -> /GPIO2
- A1 pad 21: /GPIO3 -> /GPIO6
- C1 pad 1: /GPIO6 -> /GPIO10
- C3 pad 1: /GPIO3 -> /GPIO6
- C4 pad 1: /GPIO10 -> /GPIO2
- C5 pad 1: /GPIO2 -> /GPIO3
- SW1 pad 2: /GPIO6 -> /GPIO10
Routing:
- net /GPIO6: track 55.0 -> 23.6 mm
- net /GPIO10: track 36.7 -> 48.4 mm, vias 0 -> 1
- net GND: track 98.6 -> 110.2 mm
- net /GPIO2: track 19.6 -> 18.7 mm
- net /GPIO3: track 25.1 -> 24.4 mm
