File: thumbs-down-hw/thumbs-down-hw.kicad_sch (KiCad schematic)
At the start: 26 parts, among them SW10 SW_Push, SW2 SW_Push, SW3 SW_Push, SW9 SW_Push, U1 PicoW, U2 RFM69HCW

Commit message: add thumbs-down-hw r1 gerbers
Parts:
- renumbered D2 to D1, SW2 to SW1
Connections:
- net GPIO10: now also C1.1, SW1.2; no longer A1.20 (D1), C4.1
- net GPIO2: now also A1.20 (D1), C4.1; no longer A1.19 (D0), C5.1
- net GPIO3: now also A1.19 (D0), C5.1; no longer A1.21 (D2), C3.1
- net GPIO6: now also A1.21 (D2), C3.1; no longer C1.1, SW1.2
- net LED_DI_2 renamed LED_DI_3
